File: board/board.sch (KiCad schematic (older format))
At the start: 8 parts, among them J1 Conn_01x02, P1 CONN_01X08, P2 CONN_01X08, SW1 SW_SPDT, U1 DS18B20

Commit message: Add -rescue.{lib,dcm}.
Parts:
- P1, P2: symbol board-rescue:CONN_01X08 -> board-rescue:CONN_01X08-board-rescue
Changed lines of the file:
@@
 $EndDescr
 $Comp
-L board-rescue:CONN_01X08 P1
+L board-rescue:CONN_01X08-board-rescue P1
 U 1 1 5763EB78
 P 9650 1400
@@
 $EndComp
 $Comp
-L board-rescue:CONN_01X08 P2
+L board-rescue:CONN_01X08-board-rescue P2
 U 1 1 5763EBF2
 P 10100 1400

Commit message: Switch SW1 footprint for actual part.
Parts:
- SW1: footprint (none) -> footprints:SS-12F23-SPDT
Changed lines of the file:
@@
 F 0 "SW1" H 2500 2735 50  0000 C CNN
 F 1 "SW_SPDT" H 2500 2644 50  0000 C CNN
-F 2 "" H 2500 2450 50  0001 C CNN
+F 2 "footprints:SS-12F23-SPDT" H 2500 2450 50  0001 C CNN
 F 3 "https://datasheetspdf.com/pdf-file/705135/ETC/SS-12F23-4.5/1" H 2500 2450 50  0001 C CNN
 	1    2500 2450
